File: Project1-1.kicad_sch (KiCad schematic)
At the start: 34 parts, among them IC1 LM324N, U3 LM324

Commit message: Add files via upload
Parts:
- C1: value C -> 10n; footprint (none) -> Capacitor_SMD:C_0201_0603Metric
- C2: value C -> 10n; footprint (none) -> Resistor_SMD:R_0201_0603Metric
- C3, C4: footprint (none) -> Capacitor_SMD:C_0201_0603Metric
- R1, R2, R3, R4, R5, R6: footprint (none) -> Resistor_SMD:R_0201_0603Metric
Changed lines of the file:
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@@
 			)
 		)
-		(property "Footprint" ""
+		(property "Footprint" "Resistor_SMD:R_0201_0603Metric"
 			(at 46.228 39.37 90)
 			(effects
@@
 			)
 		)
-		(property "Footprint" ""
+		(property "Footprint" "Capacitor_SMD:C_0201_0603Metric"
 			(at 93.98 72.6948 0)
 			(effects
@@
 			)
 		)
-		(property "Footprint" ""
+		(property "Footprint" "Capacitor_SMD:C_0201_0603Metric"
 			(at 93.98 80.3148 0)
 			(effects
@@
 			)
 		)
-		(property "Footprint" ""
+		(property "Footprint" "Resistor_SMD:R_0201_0603Metric"
 			(at 78.232 82.55 90)
 			(effects
@@
 			)
 		)
-		(property "Footprint" ""
+		(property "Footprint" "Resistor_SMD:R_0201_0603Metric"
 			(at 96.012 77.47 90)
 			(effects
@@
 			)
 		)
-		(property "Footprint" ""
+		(property "Footprint" "Resistor_SMD:R_0201_0603Metric"
 			(at 40.64 48.768 90)
 			(effects
@@
 			)
 		)
-		(property "Value" "C"
+		(property "Value" "10n"
 			(at 54.61 41.91 90)
 			(effects
@@
 			)
 		)
-		(property "Footprint" ""
+		(property "Footprint" "Capacitor_SMD:C_0201_0603Metric"
 			(at 50.8 47.9552 0)
 			(effects
@@
 			)
 		)
-		(property "Value" "C"
+		(property "Value" "10n"
 			(at 54.61 54.61 90)
 			(effects
@@
 			)
 		)
-		(property "Footprint" ""
+		(property "Footprint" "Resistor_SMD:R_0201_0603Metric"
 			(at 58.42 58.7248 0)
 			(effects
@@
 			)
 		)
-		(property "Footprint" ""
+		(property "Footprint" "Resistor_SMD:R_0201_0603Metric"
 			(at 76.2 77.978 90)
 			(effects
@@
 			)
 		)
-		(property "Footprint" ""
+		(property "Footprint" "Resistor_SMD:R_0201_0603Metric"
 			(at 56.642 53.34 90)
 			(effects
